File: MCU.kicad_sch (KiCad schematic)
At the start: 9 parts, among them SW1 TS-1101-C-W, SW2 TS-1101-C-W, U1 ESP32-WROOM-32D

Commit message: v2
Connections:
- net MOTOR1: now also U1.26 (IO4); no longer U1.10 (IO25)
- net MOTOR2: now also U1.27 (IO16); no longer U1.11 (IO26)
- net MOTOR3: now also U1.28 (IO17); no longer U1.12 (IO27)
- net MOTOR4: now also U1.30 (IO18); no longer U1.8 (IO32)
