File: interfaces.kicad_sch (KiCad schematic)
At the start: 38 parts, among them J1 TYPE-C-31-M-12, J2 Conn_01x02, J3 Conn_01x02, J4 Conn_01x02, J5 Conn_01x02, J9 Conn_01x03, Q2 SS8050-G, Q3 SS8050-G, Q4 CJ2302, Q5 CJ2302, Q6 CJ2302, Q7 CJ2302, U14 CP2102N-Axx-xQFN28

Commit message: v2
Parts:
- Q4, Q5, Q6, Q7: value CJ2302 -> SI2300A
Connections:
- net USP_DP is gone; now on net USB_DP: J1.A6 (DP1)
- net +3.3V: no longer C21.1, C22.1, R23.1, U14.6 (VDD), U14.7 (VREGIN)
- net MOTOR1: now also R33.1; no longer R27.1
- net MOTOR2: now also R31.1; no longer R29.1
- net MOTOR3: now also R29.1; no longer R31.1
- net MOTOR4: now also R27.1; no longer R33.1
- new net +3V3: C21.1, C22.1, R23.1, U14.6 (VDD), U14.7 (VREGIN)
