File: Mk15.kicad_pcb (KiCad board)
At the start: 2 copper layers, 88 x 108 mm, 86 parts, among them J1 TYPE-C-31-M-12, J2 Conn_01x02, J3 Conn_01x02, J4 Conn_01x02, J5 Conn_01x02, J6 Conn_01x02, J8 Conn_01x02, J9 Conn_01x03, Q1 FS8205, Q2 SS8050-G, Q3 SS8050-G, Q4 CJ2302, Q5 CJ2302, Q6 CJ2302, Q7 CJ2302, SW1 TS-1101-C-W, SW2 TS-1101-C-W, U1 ESP32-WROOM-32D, U10 TP4056, U11 DW01A, U12 SPX3819M5-L-3-3, U13 SPX3819M5-L-3-3, U14 CP2102N-Axx-xQFN28, U2 BMI088, U3 VL53L0, U6 QMC5883L, U8 BMP280

Commit message: v1-correction
Changed lines of the file:
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@@
       (effects (font (size 1 1) (thickness 0.15)))
     )
-    (fp_text value "TYPE-C-31-M-12" (at 6.43 4.135) (layer "F.Fab")
+    (fp_text value "TYPE-C-31-M-12" (at 6.43 4.135) (layer "F.Fab") hide
       (effects (font (size 1 1) (thickness 0.15)))
     )
@@
       )
     )
+  )
+  (zone (net 2) (net_name "GND") (layer "F.Cu") (hatch edge 0.508)
+    (connect_pads yes (clearance 0.254))
+    (min_thickness 0.254) (filled_areas_thickness no)
+    (fill yes (thermal_gap 0.508) (thermal_bridge_width 0.508))
+    (polygon
+      (pts
+        (xy 132.588 113.03)
+        (xy 130.048 113.03)
+        (xy 130.048 107.95)
+        (xy 132.588 107.95)
+      )
+    )

Commit message: v2
Parts:
- added C8: 10uF, Capacitor_SMD:C_0805_2012Metric_Pad1.18x1.45mm_HandSolder, F.Cu at (123.7, 69.6)
- added U4: SPX3819M5-L-3-3, Package_TO_SOT_SMD:SOT-23-5, F.Cu at (123.7, 74.2)
- C10, C14, C20, C21, C22, C23, C6, C7, C9, D1, D2, R10, R16, R22, R23, R24, R32, R33, R37, R9: moved to F.Cu
- C16, D5, U1, U12, U14: moved to B.Cu
- Q4, Q5, Q6, Q7: value CJ2302 -> SI2300A
- R2, R3, R4, R5: footprint Resistor_SMD:R_0805_2012Metric_Pad1.20x1.40mm_HandSolder -> Resistor_SMD:R_0603_1608Metric_Pad0.98x0.95mm_HandSolder
- moved J3 72.0 mm to (106.2, 99.5), turned to 90 degrees
- moved J4 68.2 mm to (106.2, 95.1), turned to 90 degrees
- moved D7 64.1 mm to (112.3, 101.1), turned to -90 degrees
- moved D8 58.7 mm to (112.3, 96.5), turned to -90 degrees
- moved Q5 50.7 mm to (116.6, 99.6), turned to 0 degrees
- moved Q6 49.9 mm to (116.6, 95.2), turned to 0 degrees
- moved R32 47.5 mm to (119.9, 95.2), turned to 90 degrees
- moved R30 45.7 mm to (119.9, 99.6), turned to 90 degrees
- moved C9 45.5 mm to (128.8, 83.0), turned to 90 degrees
- moved C10 42.0 mm to (132.3, 82.7), turned to -90 degrees
- moved R31 41.7 mm to (122.2, 95.2), turned to 90 degrees
- moved J5 41.6 mm to (106.2, 90.8), turned to 90 degrees
- moved D9 40.5 mm to (112.3, 91.9), turned to -90 degrees
- moved R29 40.3 mm to (122.2, 99.6), turned to 90 degrees
- moved U12 37.6 mm to (133.8, 109.6), turned to 180 degrees
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Connections:
- C19 pad 2: +3.3V -> +3V3
- C21 pad 1: +3.3V -> +3V3
- C22 pad 1: +3.3V -> +3V3
- J1 pad A6: USP_DP -> USB_DP
- R23 pad 1: +3.3V -> +3V3
- R27 pad 1: MOTOR1 -> MOTOR4
- R29 pad 1: MOTOR2 -> MOTOR3
- R31 pad 1: MOTOR3 -> MOTOR2
- R33 pad 1: MOTOR4 -> MOTOR1
- U1 pad 10: MOTOR1 -> unconnected-(U1-Pad10)
- U1 pad 11: MOTOR2 -> unconnected-(U1-Pad11)
- U1 pad 12: MOTOR3 -> unconnected-(U1-Pad12)
- U1 pad 26: unconnected-(U1-Pad26) -> MOTOR1
- U1 pad 27: unconnected-(U1-Pad27) -> MOTOR2
- U1 pad 28: unconnected-(U1-Pad28) -> MOTOR3
- U1 pad 30: unconnected-(U1-Pad30) -> MOTOR4
- U1 pad 8: MOTOR4 -> unconnected-(U1-Pad8)
- U12 pad 5: +3.3V -> +3V3
- U14 pad 6: +3.3V -> +3V3
- U14 pad 7: +3.3V -> +3V3
Routing:
- net VCC: track 317.6 -> 201.8 mm, vias 5 -> 7
- net +3.3V: track 205.6 -> 112.7 mm, vias 9 -> 5
- net GND: track 508.8 -> 435.8 mm, vias 26 -> 37
- net MOTOR3: track 90.7 -> 39.3 mm, vias 2 -> 3
- net MOTOR1: track 63.8 -> 22.9 mm, vias 2 -> 3
- net RTS: track 44.2 -> 80.8 mm, vias 2 -> 3
- net SCL: track 89.6 -> 60.8 mm, vias 2 -> 3
- net MOTOR4: track 19.0 -> 47.7 mm, vias 1 -> 3
- net USB_5V: track 36.0 -> 64.5 mm, vias 3 -> 4
- net DTR: track 55.8 -> 79.4 mm, vias 2 -> 1
- net +3V3: track 0.00 -> 22.1 mm, vias 0 -> 3
- net BOOT0: track 27.2 -> 49.0 mm, vias 0 -> 2
- net EN: track 34.8 -> 52.8 mm, vias 2 -> 6
- net SDA: track 78.2 -> 65.0 mm, vias 3 -> 5
- net Net-(Q7-Pad1): track 16.8 -> 6.55 mm, vias 1 -> 0
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
Commit message: board ver1.0
Routing:
- net GND: vias 37 -> 46
Other:
- board size 88 x 108 mm -> 100 x 95 mm
